File: other/BPY/Kits/Ravel/Schematic.kicad_sch (KiCad schematic)
At the start: 5 parts, among them U1 ESP32-C3_SUPERMINI

Commit message: 20/07/2026 21:04:34
Parts:
- added Lower, Upper: Motor_Servo, symbol Motor:Motor_Servo
- renumbered U1 to Ravel, D1 to Ring
Connections:
- net at Ravel.0 (GPIO0): now also Upper.1 (PWM)
- net at Ravel.1 (GPIO1): now also Lower.1 (PWM)
- net at Ravel.10 (GPIO10): now also I2C_1.4 (SDA)
- net at I2C_2.2 (VCC), Ravel.5V, Ring.1 (5V): now also Lower.2 (+), Upper.2 (+)
- net at Ravel.8 (GPIO8): no longer I2C_1.4 (SDA)
- net at BZ1.2 (-), I2C_1.1 (GND), I2C_2.1 (GND)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: now also Lower.3 (-), Upper.3 (-)
Other:
- moved on the sheet: BZ1, I2C_1, I2C_2, Ring

Commit message: 20/07/2026 21:25:38
Other:
- note added: "SSD1306"
- note removed: "SH1106"
Changed lines of the file:
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@@
 		)
 	)
-	(text "SH1106"
+	(text "SSD1306"
 		(exclude_from_sim no)
 		(at 169.926 88.138 0)
